Commit message: left arm visible group state

File: baxter/baxter_moveit_config/config/baxter_base.srdf.xacro (robot description, xacro)
@@ -36,9 +36,18 @@
         <joint name="left_e0" value="0" />
         <joint name="left_e1" value="0.75" />
-        <joint name="left_s0" value="0" />
+        <joint name="left_s0" value="-0.25" />
         <joint name="left_s1" value="-0.55" />
         <joint name="left_w0" value="0" />
         <joint name="left_w1" value="1.26" />
         <joint name="left_w2" value="0" />
+    </group_state>
+    <group_state name="left_visible" group="left_arm">
+        <joint name="left_e0" value="-0.25" />
+        <joint name="left_e1" value="0.5" />
+        <joint name="left_s0" value="-0.25" />
+        <joint name="left_s1" value="-0.48" />
+        <joint name="left_w0" value="-0.21" />
+        <joint name="left_w1" value="1.28" />
+        <joint name="left_w2" value="1.75" />
     </group_state>
     <group_state name="right_neutral" group="right_arm">
@@ -53,7 +62,7 @@
     <!--END EFFECTOR: Purpose: Represent information about an end effector.-->
      <!--VIRTUAL JOINT: Purpose: this element defines a virtual joint between a robot link and an external frame of reference (considered fixed with respect to the robot)-->
-    <virtual_joint name="world_joint" type="floating" parent_frame="world" child_link="base" />
+    <!-- <virtual_joint name="world_joint" type="floating" parent_frame="world" child_link="base" /> -->
     <!--PASSIVE JOINT: Purpose: this element is used to mark joints that are not actuated-->
-    <passive_joint name="world_joint" />
+    <!-- <passive_joint name="world_joint" /> -->
     <!--DISABLE COLLISIONS: By default it is assumed that any link of the robot could potentially come into collision with any other link in the robot. This tag disables collision checking between a specified pair of links. -->
     <disable_collisions link1="collision_head_link_1" link2="collision_head_link_2" reason="Adjacent" />

Commit message: left visible pose update

File: baxter/baxter_moveit_config/config/baxter_base.srdf.xacro (robot description, xacro)
@@ -43,5 +43,5 @@
     </group_state>
     <group_state name="left_visible" group="left_arm">
-        <joint name="left_e0" value="-0.25" />
+        <joint name="left_e0" value="-0.35" />
         <joint name="left_e1" value="0.5" />
         <joint name="left_s0" value="-0.25" />

Commit message: left_visible position changed

File: baxter/baxter_moveit_config/config/baxter_base.srdf.xacro (robot description, xacro)
@@ -43,11 +43,11 @@
     </group_state>
     <group_state name="left_visible" group="left_arm">
-        <joint name="left_e0" value="-0.35" />
-        <joint name="left_e1" value="0.5" />
-        <joint name="left_s0" value="-0.25" />
-        <joint name="left_s1" value="-0.48" />
-        <joint name="left_w0" value="-0.21" />
-        <joint name="left_w1" value="1.28" />
-        <joint name="left_w2" value="1.75" />
+        <joint name="left_e0" value="0.014" />
+        <joint name="left_e1" value="0.788" />
+        <joint name="left_s0" value="-0.366" />
+        <joint name="left_s1" value="-0.408" />
+        <joint name="left_w0" value="-0.728" />
+        <joint name="left_w1" value="1.092" />
+        <joint name="left_w2" value="1.639" />
     </group_state>
     <group_state name="right_neutral" group="right_arm">

Commit message: left_visible position changed

File: baxter/baxter_moveit_config/config/baxter_base.srdf.xacro (robot description, xacro)
@@ -43,11 +43,12 @@
     </group_state>
     <group_state name="left_visible" group="left_arm">
-        <joint name="left_e0" value="0.014" />
-        <joint name="left_e1" value="0.788" />
-        <joint name="left_s0" value="-0.366" />
-        <joint name="left_s1" value="-0.408" />
-        <joint name="left_w0" value="-0.728" />
-        <joint name="left_w1" value="1.092" />
-        <joint name="left_w2" value="1.639" />
+    0.07171360175170899, 0.8045729223266602, -0.4375680192443848, -0.3555000471862793, -0.7428301956848145, 0.9353447843444825, 1.7472041154052735
+        <joint name="left_e0" value="0.0717" />
+        <joint name="left_e1" value="0.8045" />
+        <joint name="left_s0" value="-0.4375" />
+        <joint name="left_s1" value="-0.3555" />
+        <joint name="left_w0" value="-0.7428" />
+        <joint name="left_w1" value="0.9353" />
+        <joint name="left_w2" value="1.7472" />
     </group_state>
     <group_state name="right_neutral" group="right_arm">

Commit message: new setup

File: baxter/baxter_moveit_config/config/baxter_base.srdf.xacro (robot description, xacro)
@@ -34,21 +34,23 @@
     <!--GROUP STATES: Purpose: Define a named state for a particular group, in terms of joint values. This is useful to define states like 'folded arms'-->
     <group_state name="left_neutral" group="left_arm">
-        <joint name="left_e0" value="0" />
-        <joint name="left_e1" value="0.75" />
-        <joint name="left_s0" value="-0.25" />
-        <joint name="left_s1" value="-0.55" />
-        <joint name="left_w0" value="0" />
-        <joint name="left_w1" value="1.26" />
-        <joint name="left_w2" value="0" />
+    <!-- 0.17449031442260743, 1.0408059633911133, -0.18676216071166993, -0.904281673425293, -0.6979612576904297, 1.464951650756836, 1.6156652629943848 -->
+        <joint name="left_e0" value="0.1744" />
+        <joint name="left_e1" value="1.0408" />
+        <joint name="left_s0" value="-0.1867" />
+        <joint name="left_s1" value="-0.9042" />
+        <joint name="left_w0" value="-0.6979" />
+        <joint name="left_w1" value="1.4649" />
+        <joint name="left_w2" value="1.6156" />
     </group_state>
     <group_state name="left_visible" group="left_arm">
-    0.07171360175170899, 0.8045729223266602, -0.4375680192443848, -0.3555000471862793, -0.7428301956848145, 0.9353447843444825, 1.7472041154052735
-        <joint name="left_e0" value="0.0717" />
-        <joint name="left_e1" value="0.8045" />
-        <joint name="left_s0" value="-0.4375" />
-        <joint name="left_s1" value="-0.3555" />
-        <joint name="left_w0" value="-0.7428" />
-        <joint name="left_w1" value="0.9353" />
-        <joint name="left_w2" value="1.7472" />
+    <!-- 0.09472331354370118, 1.0411894585876464, -0.4252961729553223, -0.6408204734069824, -1.0925778149230958, 1.0032234341308595, 2.0302235704467773 -->
+    <!-- 0.1100631214050293, 1.967330358215332, -0.14266021311035157, -0.9123350725524902, -0.9587379913330079, 1.3322623127563478, 2.7055586115417483 -->
+        <joint name="left_e0" value="0.1100" />
+        <joint name="left_e1" value="1.9673" />
+        <joint name="left_s0" value="-0.1426" />
+        <joint name="left_s1" value="-0.9123" />
+        <joint name="left_w0" value="-0.9587" />
+        <joint name="left_w1" value="1.3322" />
+        <joint name="left_w2" value="2.7055" />
     </group_state>
     <group_state name="right_neutral" group="right_arm">

Commit message: right arm camera top

File: baxter/baxter_moveit_config/config/baxter_base.srdf.xacro (robot description, xacro)
@@ -46,11 +46,12 @@
     <!-- 0.09472331354370118, 1.0411894585876464, -0.4252961729553223, -0.6408204734069824, -1.0925778149230958, 1.0032234341308595, 2.0302235704467773 -->
     <!-- 0.1100631214050293, 1.967330358215332, -0.14266021311035157, -0.9123350725524902, -0.9587379913330079, 1.3322623127563478, 2.7055586115417483 -->
-        <joint name="left_e0" value="0.1100" />
-        <joint name="left_e1" value="1.9673" />
-        <joint name="left_s0" value="-0.1426" />
-        <joint name="left_s1" value="-0.9123" />
-        <joint name="left_w0" value="-0.9587" />
-        <joint name="left_w1" value="1.3322" />
-        <joint name="left_w2" value="2.7055" />
+    <!-- 0.09510680874023437, 1.359106976513672, -0.39269908125, -0.9157865293212891, -0.7489661188293457, 1.3955390201843263, 2.0919662970886233 -->
+        <joint name="left_e0" value="0.0951" />
+        <joint name="left_e1" value="1.3591" />
+        <joint name="left_s0" value="-0.3926" />
+        <joint name="left_s1" value="-0.9157" />
+        <joint name="left_w0" value="-0.7489" />
+        <joint name="left_w1" value="1.3955" />
+        <joint name="left_w2" value="2.0919" />
     </group_state>
     <group_state name="right_neutral" group="right_arm">
@@ -62,4 +63,14 @@
         <joint name="right_w1" value="1.26" />
         <joint name="right_w2" value="0" />
+    </group_state>
+    <group_state name="right_top_camera" group="right_arm">
+    <!-- 0.5434126934875488, 0.7451311668640137, -0.2185922620239258, -1.4269856263000489, 0.4402524856201172, 2.086213869140625, -0.4061214131286621 -->
+        <joint name="right_e0" value="0.5434" />
+        <joint name="right_e1" value="0.7451" />
+        <joint name="right_s0" value="-0.2185" />
+        <joint name="right_s1" value="-1.4269" />
+        <joint name="right_w0" value="0.4402" />
+        <joint name="right_w1" value="2.0862" />
+        <joint name="right_w2" value="-0.4061" />
     </group_state>
     <!--END EFFECTOR: Purpose: Represent information about an end effector.-->
